File: hardware_eagle/NiceClock.brd (EAGLE design)
At the start: 197.9 x 197.9 mm, 1 part, among them IC1 LM317MSTT3

Commit message: kicad updates
Parts:
- added 8MHZ: (no value), crystal:HC49UP
- added C1, C3, C4, C5, C6, C7: 100n, rcl:C0603
- added C2: 10u, rcl:C/6032-28W
- added C8, C9: 20p, rcl:C0603
- added JP1: (no value), pinhead:1X04/90
- added R1: 400, rcl:R0603
- added R2: 240, rcl:R0603
- added R3: 100k, rcl:R0603
- IC1: value LM317MSTT3 -> LM317EMP
Connections:
- new net +3V3: C2.+, C4.1, C5.1, C6.1, C7.1, IC1.4, JP1.1, R2.2, R3.2
- new net +5V: C1.1, IC1.3
- new net GND: C1.2, C2.-, C3.2, C4.2, C5.2, C6.2, C7.2, C8.1, C9.1, JP1.4, R1.1
- new net N$1: IC1.1, R1.2, R2.1
- new net N$3: 8MHZ.1, C9.2
- new net N$4: 8MHZ.2, C8.2
- new net NRST: C3.1, R3.1
- new net SWCLK: JP1.3
- new net SWDIO: JP1.2
Changed lines of the file:
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@@
 </autorouter>
 <elements>
-<element name="IC1" library="v-reg" package="SOT223" value="LM317MSTT3" x="-5.08" y="5.08"/>
+<element name="IC1" library="v-reg" package="SOT223" value="LM317EMP" x="-5.08" y="5.08"/>
+<element name="R1" library="rcl" package="R0603" value="400" x="-5.08" y="-2.54"/>
+<element name="R2" library="rcl" package="R0603" value="240" x="-5.08" y="-7.62"/>
+<element name="C1" library="rcl" package="C0603" value="100n" x="-5.08" y="-12.7"/>
+<element name="C2" library="rcl" package="C/6032-28W" value="10u" x="-2.54" y="-17.78"/>
+<element name="JP1" library="pinhead" package="1X04/90" value="" x="0" y="-30.48"/>
+<element name="C3" library="rcl" package="C0603" value="100n" x="-5.08" y="-40.64"/>
+<element name="C4" library="rcl" package="C0603" value="100n" x="-5.08" y="-45.72"/>
+<element name="C5" library="rcl" package="C0603" value="100n" x="-5.08" y="-50.8"/>
+<element name="C6" library="rcl" package="C0603" value="100n" x="-5.08" y="-55.88"/>
+<element name="C7" library="rcl" package="C0603" value="100n" x="-5.08" y="-60.96"/>
+<element name="R3" library="rcl" package="R0603" value="100k" x="-5.08" y="-66.04"/>
+<element name="8MHZ" library="crystal" package="HC49UP" value="" x="0" y="-73.66">
+<attribute name="OC_NEWARK" value="unknown" x="0" y="-73.66" size="1.778" layer="27" display="off"/>
+<attribute name="MPN" value="" x="0" y="-73.66" size="1.778" layer="27" display="off"/>
+<attribute name="MF" value="" x="0" y="-73.66" size="1.778" layer="27" display="off"/>
+<attribute name="OC_FARNELL" value="unknown" x="0" y="-73.66" size="1.778" layer="27" display="off"/>
+</element>
+<element name="C8" library="rcl" package="C0603" value="20p" x="-5.08" y="-81.28"/>
+<element name="C9" library="rcl" package="C0603" value="20p" x="-5.08" y="-86.36"/>
 </elements>
 <signals>
+<signal name="+5V">
+<contactref element="C1" pad="1"/>
+<contactref element="IC1" pad="3"/>
+<wire x1="-2.78" y1="1.93" x2="-5.93" y2="-12.7" width="0" layer="19" extent="1-1"/>
+</signal>
+<signal name="GND">
+<contactref element="C1" pad="2"/>
+<contactref element="R1" pad="1"/>
+<contactref element="C2" pad="-"/>
+<contactref element="JP1" pad="4"/>
+<contactref element="C7" pad="2"/>
+<contactref element="C6" pad="2"/>
+<contactref element="C5" pad="2"/>
+<contactref element="C4" pad="2"/>
+<contactref element="C3" pad="2"/>
+<contactref element="C8" pad="1"/>
+<contactref element="C9" pad="1"/>
+<wire x1="-5.93" y1="-81.28" x2="-5.93" y2="-86.36" width="0" layer="19" extent="1-1"/>
+<wire x1="-4.23" y1="-60.96" x2="-5.93" y2="-81.28" width="0" layer="19" extent="1-1"/>
+<wire x1="-4.23" y1="-55.88" x2="-4.23" y2="-60.96" width="0" layer="19" extent="1-1"/>
+<wire x1="-4.23" y1="-50.8" x2="-4.23" y2="-55.88" width="0" layer="19" extent="1-1"/>
+<wire x1="-4.23" y1="-45.72" x2="-4.23" y2="-50.8" width="0" layer="19" extent="1-1"/>
+<wire x1="-4.23" y1="-40.64" x2="-4.23" y2="-45.72" width="0" layer="19" extent="1-1"/>
+<wire x1="3.81" y1="-34.29" x2="-4.23" y2="-40.64" width="0" layer="19" extent="1-1"/>
+<wire x1="-5.165" y1="-17.78" x2="3.81" y2="-34.29" width="0" layer="19" extent="1-1"/>
+<wire x1="-4.23" y1="-12.7" x2="-5.165" y2="-17.78" width="0" layer="19" extent="1-1"/>
+<wire x1="-5.93" y1="-2.54" x2="-4.23" y2="-12.7" width="0" layer="19" extent="1-1"/>
+</signal>
+<signal name="N$1">
+<contactref element="R1" pad="2"/>
+<contactref element="IC1" pad="1"/>
+<contactref element="R2" pad="1"/>
+<wire x1="-4.23" y1="-2.54" x2="-5.93" y2="-7.62" width="0" layer="19" extent="1-1"/>
+<wire x1="-7.38" y1="1.93" x2="-4.23" y2="-2.54" width="0" layer="19" extent="1-1"/>
+</signal>
+<signal name="+3V3">
+<contactref element="C2" pad="+"/>
+<contactref element="IC1" pad="4"/>
+<contactref element="R2" pad="2"/>
+<contactref element="JP1" pad="1"/>
+<contactref element="C7" pad="1"/>
+<contactref element="C6" pad="1"/>
+<contactref element="C5" pad="1"/>
+<contactref element="C4" pad="1"/>
+<contactref element="R3" pad="2"/>
+<wire x1="-5.93" y1="-60.96" x2="-4.23" y2="-66.04" width="0" layer="19" extent="1-1"/>
+<wire x1="-5.93" y1="-55.88" x2="-5.93" y2="-60.96" width="0" layer="19" extent="1-1"/>
+<wire x1="-5.93" y1="-50.8" x2="-5.93" y2="-55.88" width="0" layer="19" extent="1-1"/>
+<wire x1="-5.93" y1="-45.72" x2="-5.93" y2="-50.8" width="0" layer="19" extent="1-1"/>
+<wire x1="-3.81" y1="-34.29" x2="-5.93" y2="-45.72" width="0" layer="19" extent="1-1"/>
+<wire x1="0.085" y1="-17.78" x2="-3.81" y2="-34.29" width="0" layer="19" extent="1-1"/>
+<wire x1="-4.23" y1="-7.62" x2="0.085" y2="-17.78" width="0" layer="19" extent="1-1"/>
+<wire x1="-5.08" y1="8.23" x2="-4.23" y2="-7.62" width="0" layer="19" extent="1-1"/>
+</signal>
+<signal name="SWDIO">
+<contactref element="JP1" pad="2"/>
+</signal>
+<signal name="SWCLK">
+<contactref element="JP1" pad="3"/>
+</signal>
+<signal name="NRST">
+<contactref element="R3" pad="1"/>
+<contactref element="C3" pad="1"/>
+<wire x1="-5.93" y1="-40.64" x2="-5.93" y2="-66.04" width="0" layer="19" extent="1-1"/>
+</signal>
+<signal name="N$3">
+<contactref element="C9" pad="2"/>
+<contactref element="8MHZ" pad="1"/>
+<wire x1="-4.826" y1="-73.66" x2="-4.23" y2="-86.36" width="0" layer="19" extent="1-1"/>
+</signal>
+<signal name="N$4">
+<contactref element="C8" pad="2"/>
+<contactref element="8MHZ" pad="2"/>
+<wire x1="4.826" y1="-73.66" x2="-4.23" y2="-81.28" width="0" layer="19" extent="1-1"/>
+</signal>
 </signals>
 </board>
