File: hardware_eagle/NiceClock.sch (EAGLE design)
At the start: 1 part, among them IC1 LM317MSTT3

Commit message: kicad updates
Parts:
- added 8MHZ: (no value), crystal:CRYSTALHC49UP
- added C1, C3, C4, C5, C6, C7: 100n, rcl:C-EUC0603
- added C2: 10u, rcl:CPOL-EUC/6032-28W
- added C8, C9: 20p, rcl:C-EUC0603
- added JP1: (no value), pinhead:PINHD-1X4/90
- added R1: 400, rcl:R-EU_R0603
- added R2: 240, rcl:R-EU_R0603
- added R3: 100k, rcl:R-EU_R0603
- IC1: value LM317MSTT3 -> LM317EMP
Connections:
- new net +3V3: C2.+, C4.1, C5.1, C6.1, C7.1, IC1.OUT, JP1.1, R2.2, R3.2
- new net +5V: C1.1, IC1.IN
- new net GND: C1.2, C2.-, C3.2, C4.2, C5.2, C6.2, C7.2, C8.1, C9.1, JP1.4, R1.1
- new net N$1: IC1.ADJ, R1.2, R2.1
- new net N$3: 8MHZ.1, C9.2
- new net N$4: 8MHZ.2, C8.2
- new net NRST: C3.1, R3.1
- new net SWCLK: JP1.3
- new net SWDIO: JP1.2
