File: hardware_kicad/_autosave-NiceClock.kicad_pcb (KiCad board)
At the start: 2 copper layers, 198.2 x 198.2 mm, 294 parts, among them P1 CONN_01X04, U1 WS2811, U10 WS2811, U11 WS2811, U12 WS2811, U13 WS2811, U14 WS2811, U15 WS2811, U16 WS2811, U17 WS2811, U18 WS2811, U19 WS2811, U2 WS2811, U20 WS2811, U21 WS2811, U22 WS2811, U23 WS2811, U24 WS2811, U25 WS2811, U26 WS2811, U27 WS2811, U28 WS2811, U29 WS2811, U3 WS2811, U30 WS2811, U31 WS2811, U32 WS2811, U33 WS2811, U34 WS2811, U35 WS2811, U36 WS2811, U37 WS2811, U38 WS2811, U39 WS2811, U4 WS2811, U40 WS2811, U5 WS2811, U6 WS2811, U7 WS2811, U8 WS2811, U9 WS2811, Y1 8MHz

Commit message: kicad updates
Parts:
- moved U9 102.1 mm to (188.0, 34.3)
- moved U15 25.0 mm to (91.4, 174.0)
- moved U35 24.1 mm to (67.3, 174.0)
Routing:
- net GND: track 0.00 -> 32.3 mm
Other:
- net class Default: trace_width 2.54 -> 0.5
Changed lines of the file:
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@@
-(kicad_pcb (version 4) (host pcbnew no-vcs-found-product)
+(kicad_pcb (version 4) (host pcbnew 4.0.1-stable)
   (general
     (links 762)
-    (no_connects 336)
-    (area -53.368333 -50.567001 382.370001 294.32819)
+    (no_connects 335)
+    (area 106.564302 45.604302 304.915698 243.955698)
     (thickness 1.6)
     (drawings 8)
-    (tracks 15)
+    (tracks 20)
     (zones 0)
     (modules 294)
@@
   )
   (setup
-    (last_trace_width 2.54)
+    (last_trace_width 0.5)
     (trace_clearance 0.2)
     (zone_clearance 0.508)
@@
   (net_class Default "This is the default net class."
     (clearance 0.2)
-    (trace_width 2.54)
+    (trace_width 0.5)
     (via_dia 0.6)
     (via_drill 0.4)
@@
   )
   (module SOP8:LQFP48 (layer F.Cu)
-    (at 198.12 135.89)
+    (at 187.96 34.29)
     (fp_text reference U9 (at -5.04952 -5.00126) (layer F.SilkS)
       (effects (font (size 0.59944 0.59944) (thickness 0.12446)))
@@
   )
   (module custom_janh:SOP8 (layer F.Cu)
-    (at 104.14 195.58)
+    (at 91.44 173.99)
     (fp_text reference U15 (at -0.254 -1.016) (layer F.SilkS)
       (effects (font (thickness 0.3048)))
@@
   )
   (module custom_janh:SOP8 (layer F.Cu)
-    (at 74.93 196.85)
+    (at 67.31 173.99)
     (fp_text reference U35 (at -0.254 -1.016) (layer F.SilkS)
       (effects (font (thickness 0.3048)))
@@
   (segment (start 220.98 120.65) (end 220.98 113.03) (width 0.25) (layer F.Cu) (net 0))
   (segment (start 220.98 113.03) (end 233.68 100.33) (width 0.25) (layer F.Cu) (net 0))
+  (segment (start 71.11746 182.36946) (end 78.22946 182.36946) (width 0.5) (layer F.Cu) (net 1))
+  (segment (start 95.24746 186.69254) (end 95.24746 182.36946) (width 0.5) (layer F.Cu) (net 1))
+  (segment (start 92.71 189.23) (end 95.24746 186.69254) (width 0.5) (layer F.Cu) (net 1))
+  (segment (start 85.09 189.23) (end 92.71 189.23) (width 0.5) (layer F.Cu) (net 1))
+  (segment (start 78.22946 182.36946) (end 85.09 189.23) (width 0.5) (layer F.Cu) (net 1))
   (segment (start 255.26746 34.80054) (end 255.26746 28.10746) (width 0.25) (layer F.Cu) (net 264))
   (segment (start 255.26746 28.10746) (end 255.1 27.94) (width 0.25) (layer F.Cu) (net 264))
