File: hardware_kicad/_autosave-NiceClock.kicad_pcb (KiCad board)
At the start: 2 copper layers, 249 x 249 mm, 168 parts, among them P1 CONN_01X04, U1 WS2803, U2 WS2803, U3 WS2803, U4 WS2803, U5 WS2803, U6 WS2803, U7 WS2803, U8 STM32F101C8, U9 LM317EMP, Y1 8MHz

Commit message: some tracks and 3D drawing
Parts:
- moved C11 24.4 mm to (132.3, 160.5), turned to 90 degrees
- moved C16 19.6 mm to (127.3, 168.8), turned to 180 degrees
- moved R19 13.4 mm to (182.4, 167.4)
- moved C10 12.3 mm to (143.8, 166.9)
- moved Y1 11.2 mm to (146.3, 152.9)
- moved R17 8.89 mm to (182.4, 165.4)
- moved C8 8.64 mm to (127.3, 170.7), turned to 180 degrees
- moved C15 7.90 mm to (177.3, 162.6), turned to 270 degrees
- moved C14 6.48 mm to (185.9, 166.4), turned to 270 degrees
- moved C9 4.09 mm to (139.3, 177.0), turned to 270 degrees
Routing:
- net +3V3: track 0.00 -> 27.6 mm
- net Net-(R17-Pad1): track 0.00 -> 5.37 mm
- net +5V: track 0.00 -> 3.37 mm
- net Net-(C16-Pad1): track 0.00 -> 3.13 mm
Other:
- net class Default: trace_width 0.5 -> 0.25
