File: hardware_kicad/NiceClock.kicad_pcb (KiCad board)
At the start: 2 copper layers, 249 x 249 mm, 168 parts, among them P1 CONN_01X04, U1 WS2803, U2 WS2803, U3 WS2803, U4 WS2803, U5 WS2803, U6 WS2803, U7 WS2803, U8 STM32F101C8, U9 LM317EMP, Y1 8MHz

Commit message: pcb updates
Parts:
- added C17: 22p, Capacitors_SMD:C_0603_HandSoldering, F.Cu at (173.2, 133.6)
- added C18: 22p, Capacitors_SMD:C_0603_HandSoldering, F.Cu at (173.2, 137.7)
- added C19: 100n, Capacitors_SMD:C_0603_HandSoldering, F.Cu at (181.9, 133.1)
- added R20: 10k, Resistors_SMD:R_0603_HandSoldering, F.Cu at (185.4, 134.1)
- added R21: 2k2, Resistors_SMD:R_0603_HandSoldering, F.Cu at (187.2, 134.1)
- added R22: 2k2, Resistors_SMD:R_0603_HandSoldering, F.Cu at (189.0, 134.1)
- added U10: MCP7940M, Housings_SSOP:MSOP-8_3x3mm_Pitch0.65mm, F.Cu at (180.6, 136.3)
- added Y2: 32.768kHz, custom_janh:CRYSTAL_SMD_3.2x1.5, F.Cu at (175.5, 135.6)
- moved C11 24.4 mm to (132.3, 160.5), turned to 90 degrees
- moved C13 20.0 mm to (149.6, 149.1)
- moved C16 19.6 mm to (127.3, 168.8), turned to 180 degrees
- moved R19 13.4 mm to (182.4, 167.4)
- moved C10 12.3 mm to (143.8, 166.9)
- moved R1 12.2 mm to (181.6, 78.0), turned to 270 degrees
- moved Y1 11.2 mm to (146.3, 152.9)
- moved C1 9.91 mm to (198.9, 76.7)
- moved R17 8.89 mm to (182.4, 165.4)
- moved C8 8.64 mm to (127.3, 170.7), turned to 180 degrees
- moved C12 7.96 mm to (143.0, 149.1), turned to 180 degrees
- moved C15 7.90 mm to (177.3, 162.6), turned to 270 degrees
- moved C14 6.48 mm to (185.9, 166.4), turned to 270 degrees
- moved C9 4.09 mm to (139.3, 177.0), turned to 270 degrees
Connections:
- U8 pad 41: Net-(U8-Pad41) -> /RTC_MFP
- U8 pad 42: Net-(U8-Pad42) -> /RTC_SCL
- U8 pad 43: Net-(U8-Pad43) -> /RTC_SDA
Routing:
- net +5V: track 0.00 -> 322.1 mm
- net Net-(D1-Pad1): track 0.00 -> 69.0 mm
- net Net-(D2-Pad1): track 0.00 -> 57.6 mm
- net +3V3: track 0.00 -> 39.7 mm
- net /RTC_SDA: track 0.00 -> 7.02 mm
- net Net-(C18-Pad1): track 0.00 -> 5.75 mm
- net Net-(C17-Pad1): track 0.00 -> 5.74 mm
- net Net-(R17-Pad1): track 0.00 -> 5.37 mm
- net /RTC_SCL: track 0.00 -> 4.98 mm
- net /OSC_OUT: track 0.00 -> 4.84 mm
- net /OSC_IN: track 0.00 -> 4.84 mm
- net Net-(R1-Pad2): track 0.00 -> 3.66 mm
- net Net-(C16-Pad1): track 0.00 -> 3.13 mm
- net /RTC_MFP: track 0.00 -> 2.75 mm
Other:
- net class Default: clearance 0.2 -> 0.4; trace_width 0.5 -> 0.25
- net class power: clearance 0.2 -> 0.8
- rule trace_clearance: 0.2 -> 0.4
